Commit message: Add gazebo_plugins Edit origin positions

File: bbbot_description/urdf/bbbot.xacro (robot description, xacro)
@@ -11,12 +11,14 @@
     <origin xyz="0 0 0" rpy="0 0 0" />
   </xacro:stand>
+  <xacro:include filename="$(find manipulator_description)/urdf/common.xacro" />
+  <xacro:manipulator_arm_gazebo prefix="" />
   <!-- One of the values should be 226 mm -->
   <!-- Left arm -->
   <xacro:manipulator_h_arm prefix="leftarm" joint_limited="false" parent="world">
-    <origin xyz="0.045 0.1665 1.526" rpy="${-pi/2} 0 0" />
+    <origin xyz="0.045 0.1665 1.526" rpy="${-pi/2} ${pi/2} 0" />
   </xacro:manipulator_h_arm>
   <!-- Rsight arm -->
   <xacro:manipulator_h_arm prefix="rightarm" joint_limited="false" parent="world">
-    <origin xyz="0.045 -0.1665 1.526" rpy="${pi/2} 0 0" />
+    <origin xyz="0.045 -0.1665 1.526" rpy="${pi/2} ${pi/2} 0" />
   </xacro:manipulator_h_arm>
 </robot>

Commit message: Add fingers to the model

File: bbbot_description/urdf/bbbot.xacro (robot description, xacro)
@@ -6,4 +6,6 @@
   <!-- stand -->
   <xacro:include filename="$(find bbbot_description)/urdf/stand.xacro" />
+  <!-- fingers -->
+  <xacro:include filename="$(find bbbot_description)/urdf/fingers.xacro" />
   <!-- Used for fixing robot to Gazebo 'base_link' -->
   <link name="world"/>
@@ -19,7 +21,13 @@
     <origin xyz="0.045 0.1665 1.526" rpy="${-pi/2} ${pi/2} 0" />
   </xacro:manipulator_h_arm>
-  <!-- Rsight arm -->
+  <xacro:fingers prefix="leftarm" parent="leftarm_ee_link">
+    <origin xyz="0 0 0" rpy="0 0 0" />
+  </xacro:fingers>
+  <!-- Right arm -->
   <xacro:manipulator_h_arm prefix="rightarm" joint_limited="false" parent="world">
     <origin xyz="0.045 -0.1665 1.526" rpy="${pi/2} ${pi/2} 0" />
   </xacro:manipulator_h_arm>
+  <xacro:fingers prefix="rightarm" parent="rightarm_ee_link">
+    <origin xyz="0 0 0" rpy="0 0 0" />
+  </xacro:fingers>
 </robot>

Commit message: Fix the arm default positions to fix the new rotated positions of the arm

File: bbbot_description/urdf/bbbot.xacro (robot description, xacro)
@@ -19,5 +19,5 @@
   <!-- Left arm -->
   <xacro:manipulator_h_arm prefix="leftarm" joint_limited="false" parent="world">
-    <origin xyz="0.045 0.1665 1.526" rpy="${-pi/2} ${pi/2} 0" />
+    <origin xyz="0.045 0.1665 1.526" rpy="${-pi/2} ${-pi/2} 0" />
   </xacro:manipulator_h_arm>
   <xacro:fingers prefix="leftarm" parent="leftarm_ee_link">
@@ -26,5 +26,5 @@
   <!-- Right arm -->
   <xacro:manipulator_h_arm prefix="rightarm" joint_limited="false" parent="world">
-    <origin xyz="0.045 -0.1665 1.526" rpy="${pi/2} ${pi/2} 0" />
+    <origin xyz="0.045 -0.1665 1.526" rpy="${pi/2} ${-pi/2} 0" />
   </xacro:manipulator_h_arm>
   <xacro:fingers prefix="rightarm" parent="rightarm_ee_link">

Commit message: Use baselink instead of world as top level link

File: bbbot_description/urdf/bbbot.xacro (robot description, xacro)
@@ -9,6 +9,6 @@
   <xacro:include filename="$(find bbbot_description)/urdf/fingers.xacro" />
   <!-- Used for fixing robot to Gazebo 'base_link' -->
-  <link name="world"/>
-  <xacro:stand prefix="" parent="world">
+  <link name="base_link"/>
+  <xacro:stand prefix="" parent="base_link">
     <origin xyz="0 0 0" rpy="0 0 0" />
   </xacro:stand>
@@ -18,5 +18,5 @@
   <!-- One of the values should be 226 mm -->
   <!-- Left arm -->
-  <xacro:manipulator_h_arm prefix="leftarm" joint_limited="false" parent="world">
+  <xacro:manipulator_h_arm prefix="leftarm" joint_limited="false" parent="base_link">
     <origin xyz="0.045 0.1665 1.526" rpy="${-pi/2} ${-pi/2} 0" />
   </xacro:manipulator_h_arm>
@@ -25,5 +25,5 @@
   </xacro:fingers>
   <!-- Right arm -->
-  <xacro:manipulator_h_arm prefix="rightarm" joint_limited="false" parent="world">
+  <xacro:manipulator_h_arm prefix="rightarm" joint_limited="false" parent="base_link">
     <origin xyz="0.045 -0.1665 1.526" rpy="${pi/2} ${-pi/2} 0" />
   </xacro:manipulator_h_arm>

Commit message: Fix baselink to the world

File: bbbot_description/urdf/bbbot.xacro (robot description, xacro)
@@ -2,4 +2,5 @@
 <!-- Revolute-Revolute Manipulator -->
 <robot name="bbbot" xmlns:xacro="http://www.ros.org/wiki/xacro">
+  <xacro:arg name="gazebo" default="true"/>
   <!-- manipulator_h arm-->
   <xacro:include filename="$(find manipulator_description)/urdf/manipulator_h.xacro" />
@@ -10,4 +11,12 @@
   <!-- Used for fixing robot to Gazebo 'base_link' -->
   <link name="base_link"/>
+  <xacro:if value="$(arg gazebo)">
+    <!-- When using the pedistal, fix Baxter to Gazebo world with 'base' frame -->
+    <link name="world"/>
+    <joint name="fixed" type="fixed">
+      <parent link="world"/>
+      <child link="base_link"/>
+    </joint>
+  </xacro:if>
   <xacro:stand prefix="" parent="base_link">
     <origin xyz="0 0 0" rpy="0 0 0" />

File: bbbot_description/urdf/fingers.xacro (robot description, xacro)
@@ -25,8 +25,5 @@
         <origin xyz="0 0 0" rpy="0 0 0"/>
         <mass value="0.250"/>
-        <inertia
-            ixx="1.0" ixy="0.0" ixz="0.0"
-            iyy="1.0" iyz="0.0"
-            izz="1.0"/>
+        <inertia ixx="0.0" ixy="0.0" ixz="0.0" iyy="0.0" iyz="0.0" izz="0.0"/>
       </inertial>
     </link>

Commit message: Fix inertia related gazebo bugs

File: bbbot_description/urdf/bbbot.xacro (robot description, xacro)
@@ -2,5 +2,4 @@
 <!-- Revolute-Revolute Manipulator -->
 <robot name="bbbot" xmlns:xacro="http://www.ros.org/wiki/xacro">
-  <xacro:arg name="gazebo" default="true"/>
   <!-- manipulator_h arm-->
   <xacro:include filename="$(find manipulator_description)/urdf/manipulator_h.xacro" />
@@ -9,14 +8,5 @@
   <!-- fingers -->
   <xacro:include filename="$(find bbbot_description)/urdf/fingers.xacro" />
-  <!-- Used for fixing robot to Gazebo 'base_link' -->
   <link name="base_link"/>
-  <xacro:if value="$(arg gazebo)">
-    <!-- When using the pedistal, fix Baxter to Gazebo world with 'base' frame -->
-    <link name="world"/>
-    <joint name="fixed" type="fixed">
-      <parent link="world"/>
-      <child link="base_link"/>
-    </joint>
-  </xacro:if>
   <xacro:stand prefix="" parent="base_link">
     <origin xyz="0 0 0" rpy="0 0 0" />
@@ -27,5 +17,6 @@
   <!-- One of the values should be 226 mm -->
   <!-- Left arm -->
-  <xacro:manipulator_h_arm prefix="leftarm" joint_limited="false" parent="base_link">
+  <link name="left_base"/>
+  <xacro:manipulator_h_arm prefix="leftarm" joint_limited="false" parent="left_base">
     <origin xyz="0.045 0.1665 1.526" rpy="${-pi/2} ${-pi/2} 0" />
   </xacro:manipulator_h_arm>
@@ -34,5 +25,6 @@
   </xacro:fingers>
   <!-- Right arm -->
-  <xacro:manipulator_h_arm prefix="rightarm" joint_limited="false" parent="base_link">
+  <link name="right_base"/>
+  <xacro:manipulator_h_arm prefix="rightarm" joint_limited="false" parent="right_base">
     <origin xyz="0.045 -0.1665 1.526" rpy="${pi/2} ${-pi/2} 0" />
   </xacro:manipulator_h_arm>
@@ -40,3 +32,20 @@
     <origin xyz="0 0 0" rpy="0 0 0" />
   </xacro:fingers>
+  <!-- Merge all joints together -->
+  <link name="world" />
+  <joint name="world_left" type="fixed">
+    <parent link="world" />
+    <child link = "left_base" />
+    <origin xyz="0 0 0" rpy="0 0 0" />
+  </joint>
+  <joint name="world_right" type="fixed">
+    <parent link="world" />
+    <child link = "right_base" />
+    <origin xyz="0 0 0" rpy="0 0 0" />
+  </joint>
+  <joint name="world_stand" type="fixed">
+    <parent link="world" />
+    <child link = "base_link" />
+    <origin xyz="0 0 0" rpy="0 0 0" />
+  </joint>
 </robot>
