Commit message: Add low poly stand model

File: bbbot_description/urdf/stand.xacro (robot description, xacro)
@@ -12,4 +12,5 @@
         <geometry>
           <mesh filename="package://bbbot_description/meshes/visual/stand.stl" />
+          <!-- <mesh filename="package://bbbot_description/meshes/visual/stand_low.stl" /> -->
         </geometry>
         <material name="white"/>
