Commit message: Add material to finger and stand models

File: bbbot_description/urdf/fingers.xacro (robot description, xacro)
@@ -13,4 +13,5 @@
           <mesh filename="package://bbbot_description/meshes/visual/finger.stl" />
         </geometry>
+        <material name="white"/>
       </visual>
       <!-- Need better collision model -->

File: bbbot_description/urdf/stand.xacro (robot description, xacro)
@@ -13,4 +13,5 @@
           <mesh filename="package://bbbot_description/meshes/visual/stand.stl" />
         </geometry>
+        <material name="white"/>
       </visual>
       <collision>

Commit message: Model inertia as a box

File: bbbot_description/urdf/fingers.xacro (robot description, xacro)
@@ -21,9 +21,18 @@
           <mesh filename="package://bbbot_description/meshes/collision/finger.stl" />
         </geometry>
+        <!-- <origin xyz="0 0 0" rpy="${pi/2} 0 0"/>
+        <geometry>
+          <mesh filename="package://bbbot_description/meshes/visual/finger.stl" />
+        </geometry> -->
       </collision>
-      <inertial>
+      <!-- <inertial>
         <origin xyz="0 0 0" rpy="0 0 0"/>
         <mass value="0.250"/>
         <inertia ixx="0.0" ixy="0.0" ixz="0.0" iyy="0.0" iyz="0.0" izz="0.0"/>
+      </inertial> -->
+      <inertial>
+        <origin xyz="0 0 0.05" rpy="0 0 0"/>
+        <mass value="0.3" />
+        <inertia ixx="0.0008125" ixy="0" ixz="0" iyy="0.001125" iyz="0" izz="0.001125" />
       </inertial>
     </link>

Commit message: Fix prefix link names and modify the postioning of the collision model

File: bbbot_description/urdf/fingers.xacro (robot description, xacro)
@@ -5,7 +5,7 @@
       <xacro:insert_block name="origin" />
       <parent link="${parent}" />
-      <child link="${prefix}finger_link" />
+      <child link="${prefix}_finger_link" />
     </joint>
-    <link name="${prefix}finger_link">
+    <link name="${prefix}_finger_link">
       <visual>
         <origin xyz="0 0 0" rpy="${pi/2} 0 0"/>
@@ -17,5 +17,5 @@
       <!-- Need better collision model -->
       <collision>
-        <origin xyz="0 0 0" rpy="0 0 ${pi/2}"/>
+        <origin xyz="0 0 0" rpy="${pi/2} 0 ${pi/2}"/>
         <geometry>
           <mesh filename="package://bbbot_description/meshes/collision/finger.stl" />
